File: STM32_Environmental_Monitor_PCB.kicad_pcb (KiCad board)
At the start: 4 copper layers, 0 parts

Commit message: Complete PCB layout and pass DRC
Parts:
- added C1: 100n, Capacitor_THT:C_Disc_D4.7mm_W2.5mm_P5.00mm, F.Cu at (83.0, 106.5)
- added C2: 100n, Capacitor_THT:C_Disc_D4.7mm_W2.5mm_P5.00mm, F.Cu at (83.0, 120.5)
- added Q1: Q_NPN_EBC, STM32_Environmental_Monitor_Footprints:TO-92_Inline_P1.778mm, F.Cu at (136.0, 129.5)
- added Q2: Q_NPN_EBC, STM32_Environmental_Monitor_Footprints:TO-92_Inline_P1.778mm, F.Cu at (143.0, 129.5)
- added Q3: Q_NPN_EBC, STM32_Environmental_Monitor_Footprints:TO-92_Inline_P1.778mm, F.Cu at (150.0, 129.5)
- added Q4: Q_NPN_EBC, STM32_Environmental_Monitor_Footprints:TO-92_Inline_P1.778mm, F.Cu at (156.8, 129.4)
- added R1: 10k, Resistor_THT:R_Axial_DIN0207_L6.3mm_D2.5mm_P10.16mm_Horizontal, F.Cu at (135.4, 136.0)
- added R10: 1k, Resistor_THT:R_Axial_DIN0207_L6.3mm_D2.5mm_P10.16mm_Horizontal, F.Cu at (137.2, 113.4)
- added R11: 1k, Resistor_THT:R_Axial_DIN0207_L6.3mm_D2.5mm_P10.16mm_Horizontal, F.Cu at (144.2, 113.4)
- added R12: 1k, Resistor_THT:R_Axial_DIN0207_L6.3mm_D2.5mm_P10.16mm_Horizontal, F.Cu at (151.3, 113.4)
- added R13: 1k, Resistor_THT:R_Axial_DIN0207_L6.3mm_D2.5mm_P10.16mm_Horizontal, F.Cu at (158.0, 113.4)
- added R2: 390, Resistor_THT:R_Axial_DIN0207_L6.3mm_D2.5mm_P10.16mm_Horizontal, F.Cu at (102.0, 100.6)
- added R3: 390, Resistor_THT:R_Axial_DIN0207_L6.3mm_D2.5mm_P10.16mm_Horizontal, F.Cu at (106.5, 100.6)
- added R4: 390, Resistor_THT:R_Axial_DIN0207_L6.3mm_D2.5mm_P10.16mm_Horizontal, F.Cu at (118.9, 129.0)
- added R5: 390, Resistor_THT:R_Axial_DIN0207_L6.3mm_D2.5mm_P10.16mm_Horizontal, F.Cu at (118.9, 125.0)
- added R6: 390, Resistor_THT:R_Axial_DIN0207_L6.3mm_D2.5mm_P10.16mm_Horizontal, F.Cu at (118.9, 117.0)
- added R7: 390, Resistor_THT:R_Axial_DIN0207_L6.3mm_D2.5mm_P10.16mm_Horizontal, F.Cu at (111.0, 100.6)
- added R8: 390, Resistor_THT:R_Axial_DIN0207_L6.3mm_D2.5mm_P10.16mm_Horizontal, F.Cu at (118.9, 121.0)
- added R9: 390, Resistor_THT:R_Axial_DIN0207_L6.3mm_D2.5mm_P10.16mm_Horizontal, F.Cu at (118.9, 113.0)
- added SW1: SW_Push, Button_Switch_THT:SW_PUSH_6mm, F.Cu at (138.5, 149.0)
- added U1: NUCLEO-F303K8, STM32_Environmental_Monitor_Footprints:NUCLEO-F303K8_Socket, F.Cu at (105.6, 143.6)
- added U2: BME280-Module, STM32_Environmental_Monitor_Footprints:BME280_Module_Socket, F.Cu at (159.0, 143.5)
- added U3: CC56-12SURKWA, STM32_Environmental_Monitor_Footprints:CC56-12SURKWA_Socket, F.Cu at (135.5, 106.5)
- added U4: 74HC595, Package_DIP:DIP-16_W7.62mm_Socket, F.Cu at (90.0, 113.0)
- added U5: 74HC595, Package_DIP:DIP-16_W7.62mm_Socket, F.Cu at (90.0, 127.0)
Routing:
- net +3.3V: track 0.00 -> 155.7 mm, vias 0 -> 1
- net Net-(U1-D12): track 0.00 -> 103.2 mm, vias 0 -> 1
- net Net-(U1-D9): track 0.00 -> 102.6 mm, vias 0 -> 1
- net Net-(U1-D8): track 0.00 -> 84.2 mm
- net Net-(U4-QA): track 0.00 -> 75.2 mm
- net Net-(U1-A6): track 0.00 -> 65.6 mm, vias 0 -> 1
- net Net-(U4-QB): track 0.00 -> 64.5 mm
- net Net-(U1-D5): track 0.00 -> 59.7 mm, vias 0 -> 1
- net Net-(U1-D4): track 0.00 -> 59.4 mm, vias 0 -> 1
- net Net-(U4-QC): track 0.00 -> 54.7 mm
- net Net-(Q1-C): track 0.00 -> 52.5 mm, vias 0 -> 1
- net Net-(U5-QB): track 0.00 -> 47.2 mm, vias 0 -> 1
- net Net-(U4-QD): track 0.00 -> 44.9 mm
- net Net-(Q2-C): track 0.00 -> 43.8 mm, vias 0 -> 1
- net Net-(U3-b): track 0.00 -> 43.2 mm
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- added copper zone on B.Cu, net GND
- added copper zone on F.Cu, net GND
Other:
- board outline added: 90 x 67 mm
- copper layers 4 -> 2
- board text added: "no magic smoke pls"
