File: STM32_Environmental_Monitor_PCB.kicad_pcb (KiCad board)
At the start: 2 copper layers, 90 x 67 mm, 25 parts, among them Q1 Q_NPN_EBC, Q2 Q_NPN_EBC, Q3 Q_NPN_EBC, Q4 Q_NPN_EBC, SW1 SW_Push, U1 NUCLEO-F303K8, U2 BME280-Module, U3 CC56-12SURKWA, U4 74HC595, U5 74HC595

Commit message: Add M3 mounting holes and finalize PCB design
Parts:
- added REF**: MountingHole_3.2mm_M3, MountingHole:MountingHole_3.2mm_M3, F.Cu at (82.5, 84.5)
- added REF**: MountingHole_3.2mm_M3, MountingHole:MountingHole_3.2mm_M3, F.Cu at (165.5, 158.5)
- added REF**: MountingHole_3.2mm_M3, MountingHole:MountingHole_3.2mm_M3, F.Cu at (82.5, 158.5)
- added REF**: MountingHole_3.2mm_M3, MountingHole:MountingHole_3.2mm_M3, F.Cu at (165.5, 84.5)
Other:
- board size 90 x 67 mm -> 90 x 81 mm
