File: STM32_Environmental_Monitor_PCB.kicad_sch (KiCad schematic)
At the start: 0 parts

Commit message: Complete initial schematic design
Parts:
- added C1, C2: 100n, symbol Device:C
- added Q1, Q2, Q3, Q4: NPN, symbol Simulation_SPICE:NPN
- added R1: 10k, symbol Device:R
- added R10, R11, R12, R13: 1k, symbol Device:R
- added R2, R3, R4, R5, R6, R7, R8, R9: 390, symbol Device:R
- added SW1: SW_Push, symbol Switch:SW_Push
- added U1: NUCLEO-F303K8, symbol STM32_Environmental_Monitor_Symbols:NUCLEO-F303K8
- added U2: BME280-Module, symbol STM32_Environmental_Monitor_Symbols:BME280-Module
- added U3: CC56-12SURKWA, Display_7Segment:CA56-12SURKWA, symbol STM32_Environmental_Monitor_Symbols:CC56-12SURKWA
- added U4, U5: 74HC595, symbol 74xx:74HC595
Connections:
- new net: R13.1, U4.15 (QA)
- new net: Q4.2 (B), R13.2
- new net: R6.2, U3.1 (e)
- new net: R7.2, U3.10 (f)
- new net: R2.2, U3.11 (a)
- new net: Q1.1 (C), U3.12 (CC1)
- new net: R5.2, U3.2 (d)
- new net: R9.2, U3.3 (DPX)
- new net: R4.2, U3.4 (c)
- new net: R8.2, U3.5 (g)
- new net: Q4.1 (C), U3.6 (CC4)
- new net: R3.2, U3.7 (b)
- new net: Q3.1 (C), U3.8 (CC3)
- new net: Q2.1 (C), U3.9 (CC2)
- new net: R7.1, U5.5 (QF)
- new net: R1.2, SW1.2, U1.406 (A6)
- new net: R6.1, U5.4 (QE)
- new net: R2.1, U5.15 (QA)
- new net: R3.1, U5.1 (QB)
- new net: U1.315 (D12), U4.11 (SRCLK), U5.11 (SRCLK)
- new net: U1.312 (D9), U4.12 (RCLK), U5.12 (RCLK)
- new net: U4.9 (QH'), U5.14 (SER)
- new net: R4.1, U5.2 (QC)
- new net: R5.1, U5.3 (QD)
- new net: R8.1, U5.6 (QG)
- new net: R9.1, U5.7 (QH)
- new net: U1.308 (D5), U2.3 (SCL)
- new net: U1.307 (D4), U2.4 (SDA)
- new net: R12.1, U4.1 (QB)
- new net: Q3.2 (B), R12.2
- new net: Q2.2 (B), R11.2
- new net: U1.311 (D8), U4.14 (SER)
- new net: R11.1, U4.2 (QC)
- new net: R10.1, U4.3 (QD)
- new net: Q1.2 (B), R10.2
- new net +3.3V: C1.1, C2.1, SW1.1, U1.414 (+3V3), U2.1 (VCC), U2.5 (CSB), U4.16 (VCC), U5.16 (VCC)
- new net GND: C1.2, C2.2, Q1.3 (E), Q2.3 (E), Q3.3 (E), Q4.3 (E), R1.1, U1.402 (GND), U2.2 (GND), U4.8 (GND), U5.8 (GND)
- no-connect marks 0 -> 9

Commit message: Add custom footprints and assign component footprints
Parts:
- C1, C2: footprint (none) -> Capacitor_THT:C_Disc_D4.7mm_W2.5mm_P5.00mm
- Q1, Q2, Q3, Q4: value NPN -> Q_NPN_EBC; footprint (none) -> Package_TO_SOT_THT:TO-92_Inline; symbol Simulation_SPICE:NPN -> Transistor_BJT:Q_NPN_EBC
- R1, R10, R11, R12, R13, R2, R3, R4, R5, R6, R7, R8, R9: footprint (none) -> Resistor_THT:R_Axial_DIN0207_L6.3mm_D2.5mm_P10.16mm_Horizontal
- SW1: footprint (none) -> Button_Switch_THT:SW_PUSH_6mm
- U1: footprint (none) -> STM32_Environmental_Monitor_Footprints:NUCLEO-F303K8_Socket
- U2: footprint (none) -> STM32_Environmental_Monitor_Footprints:BME280_Module_Socket
- U3: footprint Display_7Segment:CA56-12SURKWA -> STM32_Environmental_Monitor_Footprints:CC56-12SURKWA_Socket
- U4, U5: footprint (none) -> Package_DIP:DIP-16_W7.62mm_Socket
Connections:
- net GND: now also Q1.1 (E), Q2.1 (E), Q3.1 (E), Q4.1 (E); no longer Q1.3 (E), Q2.3 (E), Q3.3 (E), Q4.3 (E)
- net at U3.12 (CC1): now also Q1.3 (C); no longer Q1.1 (C)
- net at U3.6 (CC4): now also Q4.3 (C); no longer Q4.1 (C)
- net at U3.8 (CC3): now also Q3.3 (C); no longer Q3.1 (C)
- net at U3.9 (CC2): now also Q2.3 (C); no longer Q2.1 (C)
Changed lines of the file:
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@@
 			)
 		)
-		(property "Footprint" ""
+		(property "Footprint" "Resistor_THT:R_Axial_DIN0207_L6.3mm_D2.5mm_P10.16mm_Horizontal"
 			(at 240.792 101.6 90)
 			(hide yes)
@@
 			)
 		)
-		(property "Footprint" "Display_7Segment:CA56-12SURKWA"
+		(property "Footprint" "STM32_Environmental_Monitor_Footprints:CC56-12SURKWA_Socket"
 			(at 189.23 69.85 0)
 			(hide yes)
@@
 			)
 		)
-		(property "Footprint" ""
+		(property "Footprint" "Resistor_THT:R_Axial_DIN0207_L6.3mm_D2.5mm_P10.16mm_Horizontal"
 			(at 151.13 61.468 90)
 			(hide yes)
@@
 			)
 		)
-		(property "Footprint" ""
+		(property "Footprint" "Resistor_THT:R_Axial_DIN0207_L6.3mm_D2.5mm_P10.16mm_Horizontal"
 			(at 126.492 114.3 90)
 			(hide yes)
@@
 			)
 		)
-		(property "Footprint" ""
+		(property "Footprint" "Capacitor_THT:C_Disc_D4.7mm_W2.5mm_P5.00mm"
 			(at 96.2152 60.96 0)
 			(hide yes)
@@
 			)
 		)
-		(property "Footprint" ""
+		(property "Footprint" "Resistor_THT:R_Axial_DIN0207_L6.3mm_D2.5mm_P10.16mm_Horizontal"
 			(at 151.13 58.928 90)
 			(hide yes)
@@
 			)
 		)
-		(property "Footprint" ""
+		(property "Footprint" "Resistor_THT:R_Axial_DIN0207_L6.3mm_D2.5mm_P10.16mm_Horizontal"
 			(at 151.13 48.768 90)
 			(hide yes)
@@
 			)
 		)
-		(property "Footprint" ""
+		(property "Footprint" "Package_DIP:DIP-16_W7.62mm_Socket"
 			(at 115.57 57.15 0)
 			(hide yes)
@@
 			)
 		)
-		(property "Footprint" ""
+		(property "Footprint" "STM32_Environmental_Monitor_Footprints:BME280_Module_Socket"
 			(at 151.13 129.54 0)
 			(hide yes)
@@
 			)
 		)
-		(property "Footprint" ""
+		(property "Footprint" "Resistor_THT:R_Axial_DIN0207_L6.3mm_D2.5mm_P10.16mm_Horizontal"
 			(at 223.012 101.6 90)
 			(hide yes)
@@
 	)
 	(symbol
-		(lib_id "Simulation_SPICE:NPN")
+		(lib_id "Transistor_BJT:Q_NPN_EBC")
 		(at 214.63 106.68 0)
 		(unit 1)
@@
 			)
 		)
-		(property "Value" "NPN"
+		(property "Value" "Q_NPN_EBC"
 			(at 219.71 107.9499 0)
 			(show_name no)
@@
 			)
 		)
-		(property "Footprint" ""
-			(at 278.13 106.68 0)
+		(property "Footprint" "Package_TO_SOT_THT:TO-92_Inline"
+			(at 219.71 104.14 0)
 			(hide yes)
 			(show_name no)
@@
 		)
 		(property "Datasheet" "https://ngspice.sourceforge.io/docs/ngspice-html-manual/manual.xhtml#cha_BJTs"
-			(at 278.13 106.68 0)
+			(at 214.63 106.68 0)
 			(hide yes)
 			(show_name no)
@@
 			)
 		)
-		(property "Description" "Bipolar transistor symbol for simulation only, substrate tied to the emitter"
+		(property "Description" "NPN transistor, emitter/base/collector"
 			(at 214.63 106.68 0)
 			(hide yes)
@@
 			)
 		)
-		(property "Sim.Pins" "1=C 2=B 3=E"
+		(property "Sim.Pins" "1=E 2=B 3=C"
 			(at 214.63 106.68 0)
 			(hide yes)
@@
 	)
 	(symbol
-		(lib_id "Simulation_SPICE:NPN")
+		(lib_id "Transistor_BJT:Q_NPN_EBC")
 		(at 232.41 106.68 0)
 		(unit 1)
@@
 			)
 		)
-		(property "Value" "NPN"
+		(property "Value" "Q_NPN_EBC"
 			(at 237.49 107.9499 0)
 			(show_name no)
@@
 			)
 		)
-		(property "Footprint" ""
-			(at 295.91 106.68 0)
+		(property "Footprint" "Package_TO_SOT_THT:TO-92_Inline"
+			(at 237.49 104.14 0)
 			(hide yes)
 			(show_name no)
@@
 		)
 		(property "Datasheet" "https://ngspice.sourceforge.io/docs/ngspice-html-manual/manual.xhtml#cha_BJTs"
-			(at 295.91 106.68 0)
+			(at 232.41 106.68 0)
 			(hide yes)
 			(show_name no)
@@
 			)
 		)
-		(property "Description" "Bipolar transistor symbol for simulation only, substrate tied to the emitter"
+		(property "Description" "NPN transistor, emitter/base/collector"
 			(at 232.41 106.68 0)
 			(hide yes)
@@
 			)
 		)
-		(property "Sim.Pins" "1=C 2=B 3=E"
+		(property "Sim.Pins" "1=E 2=B 3=C"
 			(at 232.41 106.68 0)
 			(hide yes)
@@
 			)
 		)
-		(property "Footprint" ""
+		(property "Footprint" "Resistor_THT:R_Axial_DIN0207_L6.3mm_D2.5mm_P10.16mm_Horizontal"
 			(at 151.13 56.388 90)
 			(hide yes)
@@
 			)
 		)
-		(property "Footprint" ""
+		(property "Footprint" "Package_DIP:DIP-16_W7.62mm_Socket"
 			(at 68.58 57.15 0)
 			(hide yes)
@@
 	)
 	(symbol
-		(lib_id "Simulation_SPICE:NPN")
+		(lib_id "Transistor_BJT:Q_NPN_EBC")
 		(at 250.19 106.68 0)
 		(unit 1)
@@
 			)
 		)
-		(property "Value" "NPN"
+		(property "Value" "Q_NPN_EBC"
 			(at 255.27 107.9499 0)
 			(show_name no)
@@
 			)
 		)
-		(property "Footprint" ""
-			(at 313.69 106.68 0)
+		(property "Footprint" "Package_TO_SOT_THT:TO-92_Inline"
+			(at 255.27 104.14 0)
 			(hide yes)
 			(show_name no)
@@
 		)
 		(property "Datasheet" "https://ngspice.sourceforge.io/docs/ngspice-html-manual/manual.xhtml#cha_BJTs"
-			(at 313.69 106.68 0)
+			(at 250.19 106.68 0)
 			(hide yes)
 			(show_name no)
@@
 			)
 		)
-		(property "Description" "Bipolar transistor symbol for simulation only, substrate tied to the emitter"
+		(property "Description" "NPN transistor, emitter/base/collector"
 			(at 250.19 106.68 0)
 			(hide yes)
@@
 			)
 		)
-		(property "Sim.Pins" "1=C 2=B 3=E"
+		(property "Sim.Pins" "1=E 2=B 3=C"
 			(at 250.19 106.68 0)
 			(hide yes)
@@
 			)
 		)
-		(property "Footprint" ""
+		(property "Footprint" "Capacitor_THT:C_Disc_D4.7mm_W2.5mm_P5.00mm"
 			(at 45.4152 60.96 0)
 			(hide yes)
@@
 			)
 		)
-		(property "Footprint" ""
+		(property "Footprint" "Resistor_THT:R_Axial_DIN0207_L6.3mm_D2.5mm_P10.16mm_Horizontal"
 			(at 151.13 51.308 90)
 			(hide yes)
@@
 			)
 		)
-		(property "Footprint" ""
+		(property "Footprint" "Resistor_THT:R_Axial_DIN0207_L6.3mm_D2.5mm_P10.16mm_Horizontal"
 			(at 187.452 101.6 90)
 			(hide yes)
@@
 			)
 		)
-		(property "Footprint" ""
+		(property "Footprint" "Resistor_THT:R_Axial_DIN0207_L6.3mm_D2.5mm_P10.16mm_Horizontal"
 			(at 151.13 64.008 90)
 			(hide yes)
@@
 			)
 		)
-		(property "Footprint" ""
+		(property "Footprint" "Resistor_THT:R_Axial_DIN0207_L6.3mm_D2.5mm_P10.16mm_Horizontal"
 			(at 205.232 101.6 90)
 			(hide yes)
@@
 			)
 		)
-		(property "Footprint" ""
+		(property "Footprint" "Button_Switch_THT:SW_PUSH_6mm"
 			(at 120.65 115.57 0)
 			(hide yes)
@@
 			)
 		)
-		(property "Footprint" ""
+		(property "Footprint" "Resistor_THT:R_Axial_DIN0207_L6.3mm_D2.5mm_P10.16mm_Horizontal"
 			(at 151.13 53.848 90)
 			(hide yes)
@@
 	)
 	(symbol
-		(lib_id "Simulation_SPICE:NPN")
+		(lib_id "Transistor_BJT:Q_NPN_EBC")
 		(at 196.85 106.68 0)
 		(unit 1)
@@
 			)
 		)
-		(property "Value" "NPN"
+		(property "Value" "Q_NPN_EBC"
 			(at 201.93 107.9499 0)
 			(show_name no)
@@
 			)
 		)
-		(property "Footprint" ""
-			(at 260.35 106.68 0)
+		(property "Footprint" "Package_TO_SOT_THT:TO-92_Inline"
+			(at 201.93 104.14 0)
 			(hide yes)
 			(show_name no)
@@
 		)
 		(property "Datasheet" "https://ngspice.sourceforge.io/docs/ngspice-html-manual/manual.xhtml#cha_BJTs"
-			(at 260.35 106.68 0)
+			(at 196.85 106.68 0)
 			(hide yes)
 			(show_name no)
@@
 			)
 		)
-		(property "Description" "Bipolar transistor symbol for simulation only, substrate tied to the emitter"
+		(property "Description" "NPN transistor, emitter/base/collector"
 			(at 196.85 106.68 0)
 			(hide yes)
@@
 			)
 		)
-		(property "Sim.Pins" "1=C 2=B 3=E"
+		(property "Sim.Pins" "1=E 2=B 3=C"
 			(at 196.85 106.68 0)
 			(hide yes)
@@
 			)
 		)
-		(property "Footprint" ""
+		(property "Footprint" "Resistor_THT:R_Axial_DIN0207_L6.3mm_D2.5mm_P10.16mm_Horizontal"
 			(at 151.13 66.548 90)
 			(hide yes)
@@
 			)
 		)
-		(property "Footprint" ""
+		(property "Footprint" "STM32_Environmental_Monitor_Footprints:NUCLEO-F303K8_Socket"
 			(at 60.96 130.81 0)
 			(hide yes)

Commit message: Complete PCB layout and pass DRC
Parts:
- Q1, Q2, Q3, Q4: footprint Package_TO_SOT_THT:TO-92_Inline -> STM32_Environmental_Monitor_Footprints:TO-92_Inline_P1.778mm
Changed lines of the file:
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@@
 			)
 		)
-		(property "Footprint" "Package_TO_SOT_THT:TO-92_Inline"
+		(property "Footprint" "STM32_Environmental_Monitor_Footprints:TO-92_Inline_P1.778mm"
 			(at 219.71 104.14 0)
 			(hide yes)
@@
 			)
 		)
-		(property "Footprint" "Package_TO_SOT_THT:TO-92_Inline"
+		(property "Footprint" "STM32_Environmental_Monitor_Footprints:TO-92_Inline_P1.778mm"
 			(at 237.49 104.14 0)
 			(hide yes)
@@
 			)
 		)
-		(property "Footprint" "Package_TO_SOT_THT:TO-92_Inline"
+		(property "Footprint" "STM32_Environmental_Monitor_Footprints:TO-92_Inline_P1.778mm"
 			(at 255.27 104.14 0)
 			(hide yes)
@@
 			)
 		)
-		(property "Footprint" "Package_TO_SOT_THT:TO-92_Inline"
+		(property "Footprint" "STM32_Environmental_Monitor_Footprints:TO-92_Inline_P1.778mm"
 			(at 201.93 104.14 0)
 			(hide yes)

Commit message: Fix 74HC595 control pins and update PCB fabrication files
Connections:
- net +3.3V: now also U4.10 (~{SRCLR}), U5.10 (~{SRCLR})
- net GND: now also U4.13 (~{OE}), U5.13 (~{OE})
- no-connect marks 9 -> 5
